File: hardware/OS-S88n.kicad_pcb (KiCad board)
At the start: 2 copper layers, 64.5 x 63.5 mm, 76 parts, among them J101 Screw_Terminal_01x03, J102 Screw_Terminal_01x03, J103 Screw_Terminal_01x03, J104 Screw_Terminal_01x03, J105 Screw_Terminal_01x03, J106 Screw_Terminal_01x03, J2101 RJ45, J2102 RJ45, Q2101 BC847, U2001 4014, U2002 4014

Commit message: made release files
Parts:
- removed G*** (x2): LOGO, custom_kicad_lib_sk:Train-Science logo small
- turned REF** to 0 degrees
Other:
- board text added: "<central"
- board text added: "S88>"
- board text removed: "<s88"
- board text removed: "central>"
